File: Hardware/KiCAD_Project_Files/BlueGiga_BLE112_XBee_Module.sch (KiCad schematic (older format))
At the start: 16 parts, among them J1 CONNECTOR_USB_TYPE_MINI_B, J2 HEADER_F_XBEE_PTH, P1 HEADER_1X8, P2 HEADER_1X3, P3 HEADER_1X8, P4 HEADER_1X2, P5 HEADER_1X10, U1 BLE112-A

Commit message: Updated Schematic to add debug header and remove unused pin headers.  PCB needs a few routes still and clean up debug header area.
Parts:
- removed J1: CONNECTOR_USB_TYPE_MINI_B, symbol CONNECTOR_USB_TYPE_MINI_B
- removed P1, P3: HEADER_1X8, symbol HEADER_1X8
- removed P2: HEADER_1X3, symbol HEADER_1X3
- removed P4: HEADER_1X2, symbol HEADER_1X2
- removed P5: HEADER_1X10, symbol HEADER_1X10
- added P1: HEADER_2X5, symbol HEADER_2X5
- gave numbers to parts that had none: 1
Connections:
- net labels added: P2_1, P2_2, VCC
- wire segments 154 -> 53
- no-connect marks 3 -> 33
Other:
- note added: "2x5 - 50MIL CC DEBUGGER CONNECTION"
- moved on the sheet: C2

Commit message: Corrected voltage regulator connections and added level shifters to inputs to BLE112.
Parts:
- removed P1: HEADER_2X5, symbol HEADER_2X5
- added P2: DEBUG, Header:HEADER_50MIL_2R10P_SMT, symbol HEADER_2x5
- added Q1, Q2, Q3: BSS138, Active:SOT-23-3_GDS, symbol MOSFET_N_BODY_DIODE_SMALL
- added R1, R2, R3, R4, R5, R6: 10k, Passive:0603, symbol RES_Small
- C1, C2, C3: footprint (none) -> Passive:C0603; Digi-Key Part# (none) -> 490-1550-1-ND
- C4, C5: value 2.2u -> 4.7u; footprint (none) -> Passive:C0603; Digi-Key Part# (none) -> 1276-2087-1-ND
- C6: footprint (none) -> Passive:C0603; Digi-Key Part# (none) -> 587-1259-1-ND
- LK1: footprint (none) -> Passive:SOLDER_LINK
- P1: renamed from J2; value HEADER_F_XBEE_PTH -> XBEE HEADER; footprint (none) -> Header:HEADER_50MIL_2R10P_SMT; Digi-Key Part# (none) -> S5800-40-ND
- U1: footprint BLE112 -> RF_Modules:BLE112; Digi-Key Part# (none) -> 1446-1017-1-ND
- U2: footprint (none) -> Active:SOT23-5_SMT; Digi-Key Part# (none) -> 863-1491-1-ND
Connections:
- net labels added: +3V3, RESET_3V3, RT_3V3, RX_3V3, VDD
- net labels removed: +3.3V, VCC
- wire segments 53 -> 77
Other:
- note added: "DEPENDING ON SUPPLY VOLTAGE TO THE XBEE MODULE:\n - BRIDGE LINK FOR 3.3V SUPPLY\n - OPEN LINK FOR 5V SUPPLY"
- note removed: "BRIDGE LINK FOR VCC = 3.3V\nOPEN LINK FOR VCC = 5V"
- moved on the sheet: C1, C2, C3, C4, C5, C6, LK1, P1, U1, U2
