File: Hardware/KiCAD_Project_Files/BlueGiga_BLE112_XBee_Module.sch (KiCad schematic (older format))
At the start: 11 parts, among them J2 HEADER_F_XBEE_PTH, P1 HEADER_2X5, U1 BLE112-A, U2 AAT3221

Commit message: Simplified design into a 3.3V-only.  A branch has been started to continue to support potential dual voltage (3.3V & 5V) designs.
Parts:
- removed LK1: SOLDER_LINK, symbol SOLDER_LINK
- removed P1: HEADER_2X5, symbol HEADER_2X5
- removed U2: AAT3221, symbol AAT3221
- added P2: DEBUG, Header:HEADER_50MIL_2R10P_SMT, symbol HEADER_2x5
- C1, C2, C3: footprint (none) -> Passive:C0603; Digi-Key Part# (none) -> 490-1550-1-ND
- C4, C5: value 2.2u -> 4.7u; footprint (none) -> Passive:C0603; Digi-Key Part# (none) -> 1276-2087-1-ND
- C6: footprint (none) -> Passive:C0603; Digi-Key Part# (none) -> 587-1259-1-ND
- P1: renamed from J2; value HEADER_F_XBEE_PTH -> XBEE HEADER; footprint (none) -> Header:HEADER_50MIL_2R10P_SMT; Digi-Key Part# (none) -> S5800-40-ND
- U1: footprint BLE112 -> RF_Modules:BLE112; Digi-Key Part# (none) -> 1446-1017-1-ND
Connections:
- net labels added: +3V3
- net labels removed: +3.3V, VCC
- wire segments 53 -> 46
- no-connect marks 33 -> 32
Other:
- note removed: "BRIDGE LINK FOR VCC = 3.3V\nOPEN LINK FOR VCC = 5V"
- moved on the sheet: C1, C2, C3, C4, C5, C6, P1, U1
